File: goose60.kicad_pcb (KiCad board)
At the start: 2 copper layers, 2 parts, among them P1 USB_C_Plug_USB2.0, U1 STM32F103CBTx

Commit message: update goose60 sch footprint
Parts:
- added C1: 22pF, Capacitor_SMD:C_0201_0603Metric, F.Cu at (-305.1, 197.5)
- added C10: 100uF/16v, Capacitor_SMD:C_0201_0603Metric, F.Cu at (-191.8, 222.8)
- added C11: 100nF/16v, Capacitor_SMD:C_0201_0603Metric, F.Cu at (-191.2, 217.2)
- added C2: 22pF, Capacitor_SMD:C_0201_0603Metric, F.Cu at (-300.8, 196.5)
- added C3: 1uF, Capacitor_SMD:C_0201_0603Metric, F.Cu at (-288.6, 214.4)
- added C4: 100nF, Capacitor_SMD:C_0201_0603Metric, F.Cu at (-284.2, 215.0)
- added C5: 100nF, Capacitor_SMD:C_0201_0603Metric, F.Cu at (-278.1, 215.1)
- added C6: 100nF, Capacitor_SMD:C_0201_0603Metric, F.Cu at (-280.4, 210.8)
- added C7: 100nF, Capacitor_SMD:C_0201_0603Metric, F.Cu at (-284.9, 210.6)
- added C8: 100nF/16v, Capacitor_SMD:C_0201_0603Metric, F.Cu at (-201.7, 228.6)
- added C9: 10uF/16v, Capacitor_SMD:C_0201_0603Metric, F.Cu at (-192.7, 228.4)
- added D1: LED, LED_SMD:LED_0805_2012Metric, F.Cu at (-278.5, 226.1)
- added D10: 1N4148, Diode_SMD:D_0603_1608Metric, F.Cu at (-282.2, 173.8)
- added D11: 1N4148, Diode_SMD:D_0603_1608Metric, F.Cu at (-278.2, 173.8)
- added D12: 1N4148, Diode_SMD:D_0603_1608Metric, F.Cu at (-286.3, 173.8)
- added D13: 1N4148, Diode_SMD:D_0603_1608Metric, F.Cu at (-262.0, 171.2)
- added D14: 1N4148, Diode_SMD:D_0603_1608Metric, F.Cu at (-257.9, 166.0)
- added D15: 1N4148, Diode_SMD:D_0603_1608Metric, F.Cu at (-294.4, 166.0)
- added D16: 1N4148, Diode_SMD:D_0603_1608Metric, F.Cu at (-278.2, 171.2)
- added D17: 1N4148, Diode_SMD:D_0603_1608Metric, F.Cu at (-266.0, 166.0)
- added D18: 1N4148, Diode_SMD:D_0603_1608Metric, F.Cu at (-278.2, 168.6)
- added D19: 1N4148, Diode_SMD:D_0603_1608Metric, F.Cu at (-290.3, 168.6)
- added D2: LED, LED_SMD:LED_0805_2012Metric, F.Cu at (-273.2, 225.8)
- added D20: 1N4148, Diode_SMD:D_0603_1608Metric, F.Cu at (-294.4, 168.6)
- added D21: 1N4148, Diode_SMD:D_0603_1608Metric, F.Cu at (-262.0, 168.6)
- added D22: 1N4148, Diode_SMD:D_0603_1608Metric, F.Cu at (-245.8, 173.8)
- added D23: 1N4148, Diode_SMD:D_0603_1608Metric, F.Cu at (-262.0, 173.8)
- added D24: 1N4148, Diode_SMD:D_0603_1608Metric, F.Cu at (-294.4, 171.2)
- added D25: 1N4148, Diode_SMD:D_0603_1608Metric, F.Cu at (-249.8, 168.6)
- added D26: 1N4148, Diode_SMD:D_0603_1608Metric, F.Cu at (-298.4, 166.0)
- added D27: 1N4148, Diode_SMD:D_0603_1608Metric, F.Cu at (-237.7, 171.2)
- added D28: 1N4148, Diode_SMD:D_0603_1608Metric, F.Cu at (-249.8, 171.2)
- added D29: 1N4148, Diode_SMD:D_0603_1608Metric, F.Cu at (-294.4, 173.8)
- added D3: LED, LED_SMD:LED_0805_2012Metric, F.Cu at (-284.9, 226.8)
- added D30: 1N4148, Diode_SMD:D_0603_1608Metric, F.Cu at (-298.4, 168.6)
- added D31: 1N4148, Diode_SMD:D_0603_1608Metric, F.Cu at (-249.8, 166.0)
- added D32: 1N4148, Diode_SMD:D_0603_1608Metric, F.Cu at (-282.2, 166.0)
- added D33: 1N4148, Diode_SMD:D_0603_1608Metric, F.Cu at (-249.8, 173.8)
- added D34: 1N4148, Diode_SMD:D_0603_1608Metric, F.Cu at (-253.9, 168.6)
- added D35: 1N4148, Diode_SMD:D_0603_1608Metric, F.Cu at (-282.2, 168.6)
- added D36: 1N4148, Diode_SMD:D_0603_1608Metric, F.Cu at (-286.3, 171.2)
- added D37: 1N4148, Diode_SMD:D_0603_1608Metric, F.Cu at (-241.7, 166.0)
- added D38: 1N4148, Diode_SMD:D_0603_1608Metric, F.Cu at (-266.0, 171.2)
- added D39: 1N4148, Diode_SMD:D_0603_1608Metric, F.Cu at (-286.3, 168.6)
- added D4: 1N4148, Diode_SMD:D_0603_1608Metric, F.Cu at (-241.7, 168.6)
- added D40: 1N4148, Diode_SMD:D_0603_1608Metric, F.Cu at (-245.8, 168.6)
- added D41: 1N4148, Diode_SMD:D_0603_1608Metric, F.Cu at (-274.1, 166.0)
- added D42: 1N4148, Diode_SMD:D_0603_1608Metric, F.Cu at (-257.9, 171.2)
- added D43: 1N4148, Diode_SMD:D_0603_1608Metric, F.Cu at (-245.8, 166.0)
- added D44: 1N4148, Diode_SMD:D_0603_1608Metric, F.Cu at (-282.2, 171.2)
- added D45: 1N4148, Diode_SMD:D_0603_1608Metric, F.Cu at (-237.7, 168.6)
- added D46: 1N4148, Diode_SMD:D_0603_1608Metric, F.Cu at (-241.7, 173.8)
- added D47: 1N4148, Diode_SMD:D_0603_1608Metric, F.Cu at (-270.1, 171.2)
- added D48: 1N4148, Diode_SMD:D_0603_1608Metric, F.Cu at (-270.1, 168.6)
- added D49: 1N4148, Diode_SMD:D_0603_1608Metric, F.Cu at (-245.8, 171.2)
- added D5: 1N4148, Diode_SMD:D_0603_1608Metric, F.Cu at (-274.1, 171.2)
- added D50: 1N4148, Diode_SMD:D_0603_1608Metric, F.Cu at (-278.2, 166.0)
- added D51: 1N4148, Diode_SMD:D_0603_1608Metric, F.Cu at (-266.0, 168.6)
- added D52: 1N4148, Diode_SMD:D_0603_1608Metric, F.Cu at (-233.6, 166.0)
- added D53: 1N4148, Diode_SMD:D_0603_1608Metric, F.Cu at (-253.9, 173.8)
- added D54: 1N4148, Diode_SMD:D_0603_1608Metric, F.Cu at (-233.6, 168.6)
- added D55: 1N4148, Diode_SMD:D_0603_1608Metric, F.Cu at (-286.3, 166.0)
- added D56: 1N4148, Diode_SMD:D_0603_1608Metric, F.Cu at (-241.7, 171.2)
- added D57: 1N4148, Diode_SMD:D_0603_1608Metric, F.Cu at (-237.7, 166.0)
- added D58: 1N4148, Diode_SMD:D_0603_1608Metric, F.Cu at (-290.3, 173.8)
- added D59: 1N4148, Diode_SMD:D_0603_1608Metric, F.Cu at (-298.4, 171.2)
- added D6: 1N4148, Diode_SMD:D_0603_1608Metric, F.Cu at (-253.9, 171.2)
- added D60: 1N4148, Diode_SMD:D_0603_1608Metric, F.Cu at (-298.4, 173.8)
- added D61: 1N4148, Diode_SMD:D_0603_1608Metric, F.Cu at (-257.9, 173.8)
- added D62: 1N4148, Diode_SMD:D_0603_1608Metric, F.Cu at (-274.1, 173.8)
- added D63: 1N4148, Diode_SMD:D_0603_1608Metric, F.Cu at (-266.0, 173.8)
- added D64: 1N4148, Diode_SMD:D_0603_1608Metric, F.Cu at (-274.1, 168.6)
- added D65: 1N4148, Diode_SMD:D_0603_1608Metric, F.Cu at (-270.1, 173.8)
- added D66: 1N4148, Diode_SMD:D_0603_1608Metric, F.Cu at (-290.3, 166.0)
- added D67: 1N4148, Diode_SMD:D_0603_1608Metric, F.Cu at (-290.3, 171.2)
- added D68: 1N4148, Diode_SMD:D_0603_1608Metric, F.Cu at (-270.1, 166.0)
- added D69: 6.3V/100V, Diode_SMD:D_SOD-323F, F.Cu at (-220.8, 214.4)
- added D7: 1N4148, Diode_SMD:D_0603_1608Metric, F.Cu at (-257.9, 168.6)
- added D70: 1SS355TE, Diode_SMD:D_SOD-323F, F.Cu at (-213.2, 211.3)
- added D8: 1N4148, Diode_SMD:D_0603_1608Metric, F.Cu at (-262.0, 166.0)
- added D9: 1N4148, Diode_SMD:D_0603_1608Metric, F.Cu at (-253.9, 166.0)
- added J1: Debugger, Connector_PinHeader_2.00mm:PinHeader_1x05_P2.00mm_Vertical, F.Cu at (-314.4, 221.2)
- added J2: USART, Connector_PinHeader_2.00mm:PinHeader_1x03_P2.00mm_Vertical, F.Cu at (-245.2, 269.7)
- added J3: SPI, Connector_PinHeader_2.00mm:PinHeader_1x05_P2.00mm_Vertical, F.Cu at (-269.2, 266.8)
- added R1: 10K, Resistor_SMD:R_0805_2012Metric, F.Cu at (-256.0, 228.9)
- added R10: 20, Resistor_SMD:R_0805_2012Metric, B.Cu at (83.2, 76.4)
- added R11: 1.5K, Resistor_SMD:R_0805_2012Metric, B.Cu at (83.9, 80.7)
- added R12: 0, Resistor_SMD:R_0805_2012Metric, F.Cu at (-309.4, 239.3)
- added R13: 0, Resistor_SMD:R_0805_2012Metric, F.Cu at (-309.3, 234.3)
- added R14: 0, Resistor_SMD:R_0805_2012Metric, F.Cu at (-308.9, 228.2)
- added R2: 10K, Resistor_SMD:R_0805_2012Metric, F.Cu at (-243.7, 228.7)
- added R3: 300, Resistor_SMD:R_0805_2012Metric, F.Cu at (-270.3, 202.9)
- added R4: 240R/5%, Resistor_SMD:R_0805_2012Metric, F.Cu at (-219.8, 229.0)
- added R5: 820R/5%, Resistor_SMD:R_0805_2012Metric, F.Cu at (-211.7, 229.0)
- added R6: 820R/5%, Resistor_SMD:R_0805_2012Metric, F.Cu at (-215.6, 220.9)
- added R7: 10K, Resistor_SMD:R_0805_2012Metric, F.Cu at (-309.4, 223.0)
- added R8: 10K, Resistor_SMD:R_0805_2012Metric, F.Cu at (-309.8, 244.8)
- added R9: 20, Resistor_SMD:R_0805_2012Metric, B.Cu at (85.8, 74.6)
- added SW1: SW_Push, Button_Switch_SMD:SW_Push_1P1T_NO_CK_KSC6xxJ, F.Cu at (-256.1, 219.2)
- added SW10: SW_Push, keyswitches:Kailh_socket_MX_optional, F.Cu at (-84.2, 65.7)
- added SW11: SW_Push, keyswitches:Kailh_socket_MX_optional, F.Cu at (-137.1, -15.0)
- added SW12: SW_Push, keyswitches:Kailh_socket_MX_optional, F.Cu at (-225.3, 49.6)
- added SW13: SW_Push, keyswitches:Kailh_socket_MX_optional, F.Cu at (-137.1, 33.4)
- added SW14: SW_Push, keyswitches:Kailh_socket_MX_optional, F.Cu at (-225.3, 65.7)
- added SW15: SW_Push, keyswitches:Kailh_socket_MX_optional, F.Cu at (-31.4, 17.3)
- added SW16: SW_Push, keyswitches:Kailh_socket_MX_optional, F.Cu at (-137.1, 17.3)
- added SW17: SW_Push, keyswitches:Kailh_socket_MX_optional, F.Cu at (-13.7, -15.0)
- added SW18: SW_Push, keyswitches:Kailh_socket_MX_optional, F.Cu at (-190.0, 81.9)
- added SW19: SW_Push, keyswitches:Kailh_socket_MX_optional, F.Cu at (-101.9, 81.9)
- added SW2: SW_Push, Button_Switch_SMD:SW_Push_1P1T_NO_CK_KSC6xxJ, F.Cu at (-242.6, 220.1)
- added SW20: SW_Push, keyswitches:Kailh_socket_MX_optional, F.Cu at (-154.8, 49.6)
- added SW21: SW_Push, keyswitches:Kailh_socket_MX_optional, F.Cu at (-190.0, 49.6)
- added SW22: SW_Push, keyswitches:Kailh_socket_MX_optional, F.Cu at (-66.6, -15.0)
- added SW23: SW_Push, keyswitches:Kailh_socket_MX_optional, F.Cu at (-225.3, 98.0)
- added SW24: SW_Push, keyswitches:Kailh_socket_MX_optional, F.Cu at (-172.4, 98.0)
- added SW25: SW_Push, keyswitches:Kailh_socket_MX_optional, F.Cu at (-190.0, -15.0)
- added SW26: SW_Push, keyswitches:Kailh_socket_MX_optional, F.Cu at (-207.7, 98.0)
- added SW27: SW_Push, keyswitches:Kailh_socket_MX_optional, F.Cu at (-207.7, 65.7)
- added SW28: SW_Push, keyswitches:Kailh_socket_MX_optional, F.Cu at (-84.2, 17.3)
- added SW29: SW_Push, keyswitches:Kailh_socket_MX_optional, F.Cu at (-13.7, 1.11)
- added SW3: SW_Push, keyswitches:Kailh_socket_MX_optional, F.Cu at (-225.3, 17.3)
- added SW30: SW_Push, keyswitches:Kailh_socket_MX_optional, F.Cu at (-101.9, 17.3)
- added SW31: SW_Push, keyswitches:Kailh_socket_MX_optional, F.Cu at (-119.5, 98.0)
- added SW32: SW_Push, keyswitches:Kailh_socket_MX_optional, F.Cu at (-154.8, 65.7)
- added SW33: SW_Push, keyswitches:Kailh_socket_MX_optional, F.Cu at (-207.7, -15.0)
- added SW34: SW_Push, keyswitches:Kailh_socket_MX_optional, F.Cu at (-84.2, 49.6)
- added SW35: SW_Push, keyswitches:Kailh_socket_MX_optional, F.Cu at (-154.8, 33.4)
- added SW36: SW_Push, keyswitches:Kailh_socket_MX_optional, F.Cu at (-66.6, 49.6)
- added SW37: SW_Push, keyswitches:Kailh_socket_MX_optional, F.Cu at (-119.5, -15.0)
- added SW38: SW_Push, keyswitches:Kailh_socket_MX_optional, F.Cu at (-66.6, 33.4)
- added SW39: SW_Push, keyswitches:Kailh_socket_MX_optional, F.Cu at (-119.5, 1.11)
- added SW4: SW_Push, keyswitches:Kailh_socket_MX_optional, F.Cu at (-154.8, 81.9)
- added SW40: SW_Push, keyswitches:Kailh_socket_MX_optional, F.Cu at (-137.1, 81.9)
- added SW41: SW_Push, keyswitches:Kailh_socket_MX_optional, F.Cu at (-225.3, 81.9)
- added SW42: SW_Push, keyswitches:Kailh_socket_MX_optional, F.Cu at (-172.4, -15.0)
- added SW43: SW_Push, keyswitches:Kailh_socket_MX_optional, F.Cu at (-225.3, 1.11)
- added SW44: SW_Push, keyswitches:Kailh_socket_MX_optional, F.Cu at (-119.5, 81.9)
- added SW45: SW_Push, keyswitches:Kailh_socket_MX_optional, F.Cu at (-190.0, 1.11)
- added SW46: SW_Push, keyswitches:Kailh_socket_MX_optional, F.Cu at (-101.9, 1.11)
- added SW47: SW_Push, keyswitches:Kailh_socket_MX_optional, F.Cu at (-31.4, 1.11)
- added SW48: SW_Push, keyswitches:Kailh_socket_MX_optional, F.Cu at (-190.0, 65.7)
- added SW49: SW_Push, keyswitches:Kailh_socket_MX_optional, F.Cu at (-66.6, 17.3)
- added SW5: SW_Push, keyswitches:Kailh_socket_MX_optional, F.Cu at (-207.7, 17.3)
- added SW50: SW_Push, keyswitches:Kailh_socket_MX_optional, F.Cu at (-172.4, 65.7)
- added SW51: SW_Push, keyswitches:Kailh_socket_MX_optional, F.Cu at (-225.3, -15.0)
- added SW52: SW_Push, keyswitches:Kailh_socket_MX_optional, F.Cu at (-172.4, 17.3)
- added SW53: SW_Push, keyswitches:Kailh_socket_MX_optional, F.Cu at (-84.2, -15.0)
- added SW54: SW_Push, keyswitches:Kailh_socket_MX_optional, F.Cu at (-49.0, 17.3)
- added SW55: SW_Push, keyswitches:Kailh_socket_MX_optional, F.Cu at (-172.4, 1.11)
- added SW56: SW_Push, keyswitches:Kailh_socket_MX_optional, F.Cu at (-225.3, 33.4)
- added SW57: SW_Push, keyswitches:Kailh_socket_MX_optional, F.Cu at (-84.2, 1.11)
- added SW58: SW_Push, keyswitches:Kailh_socket_MX_optional, F.Cu at (-66.6, 1.11)
- added SW59: SW_Push, keyswitches:Kailh_socket_MX_optional, F.Cu at (-101.9, 65.7)
- added SW6: SW_Push, keyswitches:Kailh_socket_MX_optional, F.Cu at (-31.4, -15.0)
- added SW60: SW_Push, keyswitches:Kailh_socket_MX_optional, F.Cu at (-119.5, 49.6)
- added SW61: SW_Push, keyswitches:Kailh_socket_MX_optional, F.Cu at (-154.8, 98.0)
- added SW62: SW_Push, keyswitches:Kailh_socket_MX_optional, F.Cu at (-137.1, 65.7)
- added SW63: SW_Push, keyswitches:Kailh_socket_MX_optional, F.Cu at (-207.7, 81.9)
- added SW64: SW_Push, keyswitches:Kailh_socket_MX_optional, F.Cu at (-172.4, 33.4)
- added SW65: SW_Push, keyswitches:Kailh_socket_MX_optional, F.Cu at (-190.0, 98.0)
- added SW66: SW_Push, keyswitches:Kailh_socket_MX_optional, F.Cu at (-101.9, 49.6)
- added SW67: SW_Push, keyswitches:Kailh_socket_MX_optional, F.Cu at (-154.8, -15.0)
- added SW68: SW_Push, keyswitches:Kailh_socket_MX_optional, F.Cu at (-101.9, 33.4)
- added SW69: SW_Push, keyswitches:Kailh_socket_MX_optional, F.Cu at (-172.4, 49.6)
- added SW7: SW_Push, keyswitches:Kailh_socket_MX_optional, F.Cu at (-137.1, 98.0)
- added SW70: SW_Push, keyswitches:Kailh_socket_MX_optional, F.Cu at (-190.0, 33.4)
- added SW71: SW_Push, keyswitches:Kailh_socket_MX_optional, F.Cu at (-172.4, 81.9)
- added SW72: SW_Push, keyswitches:Kailh_socket_MX_optional, F.Cu at (-49.0, 33.4)
- added SW73: SW_Push, keyswitches:Kailh_socket_MX_optional, F.Cu at (-101.9, -15.0)
- added SW74: SW_Push, keyswitches:Kailh_socket_MX_optional, F.Cu at (-137.1, 1.11)
- added SW75: SW_Push, keyswitches:Kailh_socket_MX_optional, F.Cu at (-84.2, 33.4)
- added SW76: SW_Push, keyswitches:Kailh_socket_MX_optional, F.Cu at (3.91, -15.0)
- added SW77: SW_Push, keyswitches:Kailh_socket_MX_optional, F.Cu at (-49.0, 1.11)
- added SW78: SW_Push, keyswitches:Kailh_socket_MX_optional, F.Cu at (-119.5, 33.4)
- added SW79: SW_Push, keyswitches:Kailh_socket_MX_optional, F.Cu at (-207.7, 49.6)
- added SW8: SW_Push, keyswitches:Kailh_socket_MX_optional, F.Cu at (-207.7, 1.11)
- added SW80: SW_Push, keyswitches:Kailh_socket_MX_optional, F.Cu at (-154.8, 17.3)
- added SW81: SW_Push, keyswitches:Kailh_socket_MX_optional, F.Cu at (-154.8, 1.11)
- added SW82: SW_Push, keyswitches:Kailh_socket_MX_optional, F.Cu at (-207.7, 33.4)
- added SW83: SW_Push, keyswitches:Kailh_socket_MX_optional, F.Cu at (-119.5, 17.3)
- added SW84: SW_Push, keyswitches:Kailh_socket_MX_optional, F.Cu at (-190.0, 17.3)
- added SW85: SW_Push, keyswitches:Kailh_socket_MX_optional, F.Cu at (-137.1, 49.6)
- added SW86: SW_Push, keyswitches:Kailh_socket_MX_optional, F.Cu at (-49.0, -15.0)
- added SW9: SW_Push, keyswitches:Kailh_socket_MX_optional, F.Cu at (-15.8, 58.5)
- added U2: LM317_SOT-223, Package_TO_SOT_SMD:SOT-223-3_TabPin2, F.Cu at (-203.8, 218.1)
- added X1: Crystal_GND24, Crystal:Crystal_SMD_TXC_7M-4Pin_3.2x2.5mm, F.Cu at (-301.8, 202.5)
- P1: moved to B.Cu
- moved U1 384.0 mm to (-284.0, 199.1)
- moved P1 20.4 mm to (80.7, 66.6)
Connections:
- net Net-(P1-PadA4) renamed VIN
- P1 pad A1: Net-(P1-PadA1) -> GND
- P1 pad A12: Net-(P1-PadA1) -> GND
- P1 pad A6: unconnected-(P1-PadA6) -> Net-(P1-PadA6)
- P1 pad A7: unconnected-(P1-PadA7) -> Net-(P1-PadA7)
- P1 pad B1: Net-(P1-PadA1) -> GND
- P1 pad B12: Net-(P1-PadA1) -> GND
- P1 pad S1: unconnected-(P1-PadS1) -> GND
- U1 pad 1: unconnected-(U1-Pad1) -> +3.3V
- U1 pad 11: unconnected-(U1-Pad11) -> /row5
- U1 pad 12: unconnected-(U1-Pad12) -> /row4
- U1 pad 13: unconnected-(U1-Pad13) -> /row3
- U1 pad 14: unconnected-(U1-Pad14) -> CAPS_LED
- U1 pad 15: unconnected-(U1-Pad15) -> SCK
- U1 pad 16: unconnected-(U1-Pad16) -> MISO
- U1 pad 17: unconnected-(U1-Pad17) -> MOSI
- U1 pad 18: unconnected-(U1-Pad18) -> /row2
- U1 pad 19: unconnected-(U1-Pad19) -> /row1
- U1 pad 20: unconnected-(U1-Pad20) -> /col8
- U1 pad 21: unconnected-(U1-Pad21) -> /col9
- U1 pad 22: unconnected-(U1-Pad22) -> /col10
- U1 pad 23: unconnected-(U1-Pad23) -> GND
- U1 pad 24: unconnected-(U1-Pad24) -> +3.3V
- U1 pad 25: unconnected-(U1-Pad25) -> /col11
- U1 pad 26: unconnected-(U1-Pad26) -> /col12
- U1 pad 27: unconnected-(U1-Pad27) -> /col13
- U1 pad 28: unconnected-(U1-Pad28) -> /col14
- U1 pad 30: unconnected-(U1-Pad30) -> MCU_TX
- U1 pad 31: unconnected-(U1-Pad31) -> MCU_RX
- U1 pad 32: unconnected-(U1-Pad32) -> USB_D-
- U1 pad 33: unconnected-(U1-Pad33) -> USB_D+
- U1 pad 34: unconnected-(U1-Pad34) -> SWDIO
- U1 pad 35: unconnected-(U1-Pad35) -> GND
- U1 pad 36: unconnected-(U1-Pad36) -> +3.3V
- U1 pad 37: unconnected-(U1-Pad37) -> SWCLK
- U1 pad 39: unconnected-(U1-Pad39) -> /col1
- U1 pad 40: unconnected-(U1-Pad40) -> /col2
- U1 pad 41: unconnected-(U1-Pad41) -> /col3
- U1 pad 42: unconnected-(U1-Pad42) -> /col4
- U1 pad 43: unconnected-(U1-Pad43) -> /col5
- U1 pad 44: unconnected-(U1-Pad44) -> BOOT0
- U1 pad 45: unconnected-(U1-Pad45) -> /col6
- U1 pad 46: unconnected-(U1-Pad46) -> /col7
- U1 pad 47: unconnected-(U1-Pad47) -> GND
- U1 pad 48: unconnected-(U1-Pad48) -> +3.3V
- U1 pad 5: unconnected-(U1-Pad5) -> XTAL1
- U1 pad 6: unconnected-(U1-Pad6) -> XTAL2
- U1 pad 7: unconnected-(U1-Pad7) -> RESET
- U1 pad 8: unconnected-(U1-Pad8) -> GND
- U1 pad 9: unconnected-(U1-Pad9) -> +3.3V
Other:
- board outline added: 285 x 94.6 mm
- board text added: "bottom routing path Ø 2mm"
- board text added: "top routing path Ø 2mm"
- board text added: "v-score on left side"
- board text added: "v-score on right side"

Commit message: update footpoint and add pcb layout
Parts:
- D10, D7, U1: moved to B.Cu
- R10, R11, R9: footprint Resistor_SMD:R_0805_2012Metric -> Resistor_SMD:R_0603_1608Metric
- SW10, SW11, SW12, SW13, SW14, SW15, SW16, SW17, SW18, SW19, SW20, SW21, SW22, SW23, SW24, SW25, SW26, SW27, SW28, SW29, SW3, SW30, SW31, SW32, SW33, SW34, SW35, SW36, SW37, SW38, SW39, SW4, SW40, SW41, SW42, SW43, SW44, SW45, SW46, SW47, SW48, SW49, SW5, SW50, SW51, SW52, SW53, SW54, SW55, SW56, SW57, SW58, SW59, SW6, SW60, SW61, SW62, SW63, SW64, SW65, SW66, SW67, SW68, SW69, SW7, SW70, SW71, SW72, SW73, SW74, SW75, SW76, SW77, SW78, SW79, SW8, SW80, SW81, SW82, SW83, SW84, SW85, SW86, SW9: footprint keyswitches:Kailh_socket_MX_optional -> keyswitches:Kailh_socket_MX
- moved SW84 541.7 mm to (335.1, 150.2), turned to 180 degrees
- moved SW70 536.5 mm to (337.5, 131.2)
- moved SW82 536.1 mm to (326.9, 74.2), turned to 180 degrees
- moved SW79 534.8 mm to (320.9, 131.2), turned to 180 degrees
- moved D12 510.9 mm to (180.2, -34.5)
- moved D17 510.9 mm to (200.4, -42.3)
- moved D36 510.9 mm to (180.2, -37.1)
- moved D38 510.9 mm to (200.4, -37.1)
- moved D39 510.9 mm to (180.2, -39.7)
- moved D51 510.9 mm to (200.4, -39.7)
- moved D55 510.9 mm to (180.2, -42.3)
- moved D63 510.9 mm to (200.4, -34.5)
- moved D11 510.9 mm to (188.3, -34.5)
- moved D13 510.9 mm to (204.5, -37.1)
- moved D14 510.9 mm to (208.5, -42.3)
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
Commit message: update diode location
Parts:
- D11, D12, D13, D14, D15, D16, D17, D18, D19, D20, D21, D22, D23, D24, D25, D26, D27, D28, D29, D30, D31, D32, D33, D34, D35, D36, D37, D38, D39, D4, D40, D41, D42, D43, D44, D45, D46, D47, D48, D49, D5, D50, D51, D52, D53, D54, D55, D56, D57, D58, D59, D6, D60, D61, D62, D63, D64, D65, D66, D67, D68, D8, D9: moved to B.Cu
- moved D66 241.6 mm to (327.5, 146.0), turned to 180 degrees
- moved D6 239.3 mm to (65.3, 151.5), turned to 180 degrees
- moved D60 225.1 mm to (302.5, 145.9), turned to 180 degrees
- moved D59 220.5 mm to (316.2, 126.2), turned to 180 degrees
- moved D9 215.1 mm to (112.0, 147.9), turned to 180 degrees
- moved D5 212.3 mm to (70.0, 136.3), turned to 180 degrees
- moved D4 209.3 mm to (89.0, 119.7), turned to 180 degrees
- moved D14 203.0 mm to (135.4, 147.1), turned to 180 degrees
- moved D13 202.8 mm to (101.3, 137.5), turned to 180 degrees
- moved D58 201.5 mm to (278.1, 139.2), turned to 180 degrees
- moved D65 199.3 mm to (300.4, 135.5), turned to 180 degrees
- moved D54 199.0 mm to (278.7, 153.9), turned to 180 degrees
- moved D22 198.7 mm to (126.5, 140.4), turned to 180 degrees
- moved D8 198.0 mm to (66.0, 99.3), turned to 180 degrees
- moved D18 197.2 mm to (107.3, 140.1), turned to 180 degrees
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
Commit message: remove key
Parts:
- removed D13, D48: 1N4148, Diode_SMD:D_0603_1608Metric
- removed SW12, SW13, SW17, SW19, SW33, SW34, SW4, SW55, SW57, SW6, SW63, SW64, SW70, SW72, SW77, SW8, SW81, SW83, SW85: SW_Push, keyswitches:Kailh_socket_MX
- moved SW69 33.3 mm to (337.5, 131.2)
- moved SW82 1.07 mm to (328.0, 74.2)
- moved SW5 0.78 mm to (83.4, 131.2)
- turned SW80 to 0 degrees

Commit message: update components location
Parts:
- C1, C10, C11, C2, C3, C4, C5, C6, C7, C8, C9: footprint Capacitor_SMD:C_0201_0603Metric -> Capacitor_SMD:C_0603_1608Metric; moved to B.Cu
- D69, D70: footprint Diode_SMD:D_SOD-323F -> Diode_SMD:D_0603_1608Metric; moved to B.Cu
- J1, SW1, SW2, U2, X1: moved to B.Cu
- R1, R12, R13, R14, R2, R3, R4, R5, R6, R7, R8: footprint Resistor_SMD:R_0805_2012Metric -> Resistor_SMD:R_0603_1608Metric; moved to B.Cu
- moved R1 319.5 mm to (227.1, 152.6), turned to 180 degrees
- moved SW1 314.1 mm to (222.6, 147.7), turned to 180 degrees
- moved SW2 313.1 mm to (234.9, 147.7), turned to 180 degrees
- moved R2 310.7 mm to (230.5, 152.6)
- moved C1 305.9 mm to (170.1, 152.6), turned to 45 degrees
- moved R12 302.5 mm to (144.9, 127.2), turned to -90 degrees
- moved C2 302.1 mm to (170.1, 148.8), turned to -45 degrees
- moved X1 301.3 mm to (167.6, 150.4), turned to 135 degrees
- moved R13 298.6 mm to (142.7, 127.2), turned to -90 degrees
- moved R8 298.4 mm to (137.6, 126.4)
- moved R7 298.3 mm to (144.3, 121.1), turned to 180 degrees
- moved J1 296.3 mm to (138.7, 123.8), turned to -90 degrees
- moved R14 294.1 mm to (140.7, 127.2), turned to -90 degrees
- moved C3 283.8 mm to (160.4, 148.9), turned to 45 degrees
- moved C4 280.4 mm to (160.1, 144.1), turned to 135 degrees
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
Commit message: add HOLE
Parts:
- added ?: , , F.Cu at (322.6, 93.1)
- added ?: , , F.Cu at (64.3, 121.7)
- added ?: , , F.Cu at (87.8, 93.1)
- added ?: , , F.Cu at (251.9, 150.4)
- added HOLE: VAL**, hole:PKRH, F.Cu at (223.0, 44.4)
- added HOLE: VAL**, hole:PKRHSL, F.Cu at (344.9, 121.7)
- turned SW10 to 0 degrees
- turned SW69 to 180 degrees
Changed lines of the file:
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@@
       (net 107 "/col13") (pinfunction "2") (pintype "passive"))
   )
+  (footprint "hole:PKRH" (layer "F.Cu")
+    (at 222.97 44.39)
+    (attr exclude_from_pos_files exclude_from_bom)
+    (fp_text reference "HOLE" (at 0.1753 5.7861) (layer "F.SilkS") hide
+      (effects (font (size 1.524 1.524) (thickness 0.3048)))
+    )
+    (fp_text value "VAL**" (at 0.17526 -4.9022) (layer "F.SilkS") hide
+      (effects (font (size 1.524 1.524) (thickness 0.3048)))
+    )
+    (pad "1" thru_hole circle locked (at 0 0) (size 7.00024 7.00024) (drill oval 5.00126 2.49936) (layers *.Cu *.Mask))
+    (model "cherry_mx1.wrl"
+      (offset (xyz 0 0 0))
+      (scale (xyz 1 1 1))
+      (rotate (xyz 0 0 0))
+    )
+  )
   (footprint "keyswitches:Kailh_socket_MX" (layer "F.Cu")
     (at 123.74728 112.20758 180)
@@
       (net 97 "/col3") (pinfunction "2") (pintype "passive"))
   )
+  (footprint "hole:PKRHSL" (layer "F.Cu")
+    (at 344.95 121.67)
+    (attr exclude_from_pos_files exclude_from_bom)
+    (fp_text reference "HOLE" (at 0 4.675) (layer "F.SilkS") hide
+      (effects (font (size 1.524 1.524) (thickness 0.3048)))
+    )
+    (fp_text value "VAL**" (at 0.508 -4.826) (layer "F.SilkS") hide
+      (effects (font (size 1.524 1.524) (thickness 0.3048)))
+    )
+    (pad "1" thru_hole oval locked (at 0 0) (size 9.99998 5.00126) (drill oval 7.00024 2.49936) (layers *.Cu *.Mask))
+    (model "cherry_mx1.wrl"
+      (offset (xyz 0 0 0))
+      (scale (xyz 1 1 1))
+      (rotate (xyz 0 0 0))
+    )
+  )
   (footprint "keyswitches:Kailh_socket_MX" (layer "F.Cu")
     (at 78.62251 112.20758 180)
@@
   )
   (footprint "keyswitches:Kailh_socket_MX" (layer "F.Cu")
-    (at 76.37194 93.20838 180)
+    (at 76.37194 93.20838)
     (descr "MX-style keyswitch with Kailh socket mount")
     (tags "MX,cherry,gateron,kailh,pg1511,socket")
@@
     (fp_line (start -7.5 7.5) (end -7.5 -7.5) (layer "F.Fab") (width 0.15))
     (fp_line (start 7.5 7.5) (end -7.5 7.5) (layer "F.Fab") (width 0.15))
-    (pad "" np_thru_hole circle locked (at 2.54 -5.08 180) (size 3 3) (drill 3) (layers *.Cu *.Mask))
-    (pad "" np_thru_hole circle locked (at -5.08 0 180) (size 1.7018 1.7018) (drill 1.7018) (layers *.Cu *.Mask))
-    (pad "" np_thru_hole circle locked (at 0 0 180) (size 3.9878 3.9878) (drill 3.9878) (layers *.Cu *.Mask))
-    (pad "" np_thru_hole circle locked (at 5.08 0 180) (size 1.7018 1.7018) (drill 1.7018) (layers *.Cu *.Mask))
-    (pad "" np_thru_hole circle locked (at -3.81 -2.54 180) (size 3 3) (drill 3) (layers *.Cu *.Mask))
-    (pad "1" smd rect locked (at 6.29 -5.08 180) (size 2.55 2.5) (layers "B.Cu" "B.Paste" "B.Mask")
+    (pad "" np_thru_hole circle locked (at 2.54 -5.08) (size 3 3) (drill 3) (layers *.Cu *.Mask))
+    (pad "" np_thru_hole circle locked (at -5.08 0) (size 1.7018 1.7018) (drill 1.7018) (layers *.Cu *.Mask))
+    (pad "" np_thru_hole circle locked (at 0 0) (size 3.9878 3.9878) (drill 3.9878) (layers *.Cu *.Mask))
+    (pad "" np_thru_hole circle locked (at 5.08 0) (size 1.7018 1.7018) (drill 1.7018) (layers *.Cu *.Mask))
+    (pad "" np_thru_hole circle locked (at -3.81 -2.54) (size 3 3) (drill 3) (layers *.Cu *.Mask))
+    (pad "1" smd rect locked (at 6.29 -5.08) (size 2.55 2.5) (layers "B.Cu" "B.Paste" "B.Mask")
       (net 16 "Net-(D8-Pad1)") (pinfunction "1") (pintype "passive"))
-    (pad "2" smd rect locked (at -7.56 -2.54 180) (size 2.55 2.5) (layers "B.Cu" "B.Paste" "B.Mask")
+    (pad "2" smd rect locked (at -7.56 -2.54) (size 2.55 2.5) (layers "B.Cu" "B.Paste" "B.Mask")
       (net 95 "/col1") (pinfunction "2") (pintype "passive"))
   )
@@
       (net 108 "/col14") (pinfunction "2") (pintype "passive"))
   )
+  (footprint "" (layer "F.Cu")
+    (at 322.62 93.06)
+    (fp_text reference "" (at 0 0) (layer "F.SilkS")
+      (effects (font (size 1.27 1.27) (thickness 0.15)))
+    )
+    (fp_text value "" (at 0 0) (layer "F.SilkS")
+      (effects (font (size 1.27 1.27) (thickness 0.15)))
+    )
+    (pad "1" thru_hole circle locked (at 0 0) (size 7.00024 7.00024) (drill oval 5.00126 2.49936) (layers *.Cu *.Mask))
+  )
   (footprint "keyswitches:Kailh_socket_MX" (layer "F.Cu")
     (at 97.62425 150.20852 180)
@@
       (net 100 "/col6") (pinfunction "2") (pintype "passive"))
   )
+  (footprint "" (layer "F.Cu")
+    (at 64.35 121.7)
+    (fp_text reference "" (at 0 0) (layer "F.SilkS")
+      (effects (font (size 1.27 1.27) (thickness 0.15)))
+    )
+    (fp_text value "" (at 0 0) (layer "F.SilkS")
+      (effects (font (size 1.27 1.27) (thickness 0.15)))
+    )
+    (pad "1" thru_hole oval locked (at 0 0) (size 9.99998 5.00126) (drill oval 7.00024 2.49936) (layers *.Cu *.Mask))
+  )
   (footprint "LED_SMD:LED_0805_2012Metric" (layer "F.Cu")
     (at 78.55 103.02)
@@
       (net 97 "/col3") (pinfunction "2") (pintype "passive"))
   )
+  (footprint "" (layer "F.Cu")
+    (at 87.75 93.08)
+    (fp_text reference "" (at 0 0) (layer "F.SilkS")
+      (effects (font (size 1.27 1.27) (thickness 0.15)))
+    )
+    (fp_text value "" (at 0 0) (layer "F.SilkS")
+      (effects (font (size 1.27 1.27) (thickness 0.15)))
+    )
+    (pad "1" thru_hole circle locked (at 0 0) (size 7.0013 7.0013) (drill 2.4994) (layers *.Cu *.Mask))
+  )
   (footprint "keyswitches:Kailh_socket_MX" (layer "F.Cu")
     (at 118.99748 93.20838 180)
@@
   )
   (footprint "keyswitches:Kailh_socket_MX" (layer "F.Cu")
-    (at 337.50058 131.20932)
+    (at 337.50058 131.20932 180)
     (descr "MX-style keyswitch with Kailh socket mount")
     (tags "MX,cherry,gateron,kailh,pg1511,socket")
@@
     (fp_line (start -7.5 7.5) (end -7.5 -7.5) (layer "F.Fab") (width 0.15))
     (fp_line (start -7.5 -7.5) (end 7.5 -7.5) (layer "F.Fab") (width 0.15))
-    (pad "" np_thru_hole circle locked (at -3.81 -2.54) (size 3 3) (drill 3) (layers *.Cu *.Mask))
-    (pad "" np_thru_hole circle locked (at 2.54 -5.08) (size 3 3) (drill 3) (layers *.Cu *.Mask))
-    (pad "" np_thru_hole circle locked (at 0 0) (size 3.9878 3.9878) (drill 3.9878) (layers *.Cu *.Mask))
-    (pad "" np_thru_hole circle locked (at 5.08 0) (size 1.7018 1.7018) (drill 1.7018) (layers *.Cu *.Mask))
-    (pad "" np_thru_hole circle locked (at -5.08 0) (size 1.7018 1.7018) (drill 1.7018) (layers *.Cu *.Mask))
-    (pad "1" smd rect locked (at 6.29 -5.08) (size 2.55 2.5) (layers "B.Cu" "B.Paste" "B.Mask")
+    (pad "" np_thru_hole circle locked (at -3.81 -2.54 180) (size 3 3) (drill 3) (layers *.Cu *.Mask))
+    (pad "" np_thru_hole circle locked (at 2.54 -5.08 180) (size 3 3) (drill 3) (layers *.Cu *.Mask))
+    (pad "" np_thru_hole circle locked (at 0 0 180) (size 3.9878 3.9878) (drill 3.9878) (layers *.Cu *.Mask))
+    (pad "" np_thru_hole circle locked (at 5.08 0 180) (size 1.7018 1.7018) (drill 1.7018) (layers *.Cu *.Mask))
+    (pad "" np_thru_hole circle locked (at -5.08 0 180) (size 1.7018 1.7018) (drill 1.7018) (layers *.Cu *.Mask))
+    (pad "1" smd rect locked (at 6.29 -5.08 180) (size 2.55 2.5) (layers "B.Cu" "B.Paste" "B.Mask")
       (net 66 "Net-(D59-Pad1)") (pinfunction "1") (pintype "passive"))
-    (pad "2" smd rect locked (at -7.56 -2.54) (size 2.55 2.5) (layers "B.Cu" "B.Paste" "B.Mask")
+    (pad "2" smd rect locked (at -7.56 -2.54 180) (size 2.55 2.5) (layers "B.Cu" "B.Paste" "B.Mask")
       (net 107 "/col13") (pinfunction "2") (pintype "passive"))
   )
@@
       (net 103 "/col9") (pinfunction "2") (pintype "passive"))
   )
+  (footprint "" (layer "F.Cu")
+    (at 251.93 150.38)
+    (fp_text reference "" (at 0 0) (layer "F.SilkS")
+      (effects (font (size 1.27 1.27) (thickness 0.15)))
+    )
+    (fp_text value "" (at 0 0) (layer "F.SilkS")
+      (effects (font (size 1.27 1.27) (thickness 0.15)))
+    )
+    (pad "1" thru_hole circle locked (at 0 0) (size 7.00024 7.00024) (drill oval 5.00126 2.49936) (layers *.Cu *.Mask))
+  )
   (footprint "keyswitches:Kailh_socket_MX" (layer "F.Cu")

Commit message: update MX socket loaction
Parts:
- added H1: MountingHole, MountingHole:MountingHole_3.2mm_M3_Pad, F.Cu at (248.7, 36.6)
- added H2: MountingHole, MountingHole:MountingHole_3.2mm_M3_Pad, F.Cu at (240.7, 36.6)
- added H3: MountingHole, MountingHole:MountingHole_3.2mm_M3_Pad, F.Cu at (232.8, 36.6)
- added H4: MountingHole, MountingHole:MountingHole_3.2mm_M3, F.Cu at (207.3, 44.8)
- added H5: MountingHole, MountingHole:MountingHole_3.2mm_M3_Pad, F.Cu at (213.4, 36.2)
- added H6: MountingHole, MountingHole:MountingHole_3.2mm_M3_Pad, F.Cu at (223.9, 36.1)
- moved HOLE 24.0 mm to (199.0, 46.0)
- moved D63 8.83 mm to (313.4, 119.7)
- moved D1 5.37 mm to (73.0, 107.6)
- moved D3 5.28 mm to (84.6, 107.5)
- moved D2 4.54 mm to (78.8, 107.6)
- moved R3 3.16 mm to (69.1, 109.9)
- moved D64 1.49 mm to (318.1, 120.6)
- moved SW78 1.24 mm to (336.0, 103.6)
- moved SW69 0.95 mm to (338.4, 131.6), turned to 0 degrees
- moved SW79 0.91 mm to (321.7, 131.6)
- moved SW76 0.91 mm to (326.5, 112.5)
- moved SW82 0.88 mm to (328.9, 74.4)
- moved SW80 0.88 mm to (312.2, 131.6)
- moved SW75 0.88 mm to (314.6, 112.5)
- moved SW74 0.85 mm to (309.8, 93.5)
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