File: switches.kicad_sch (KiCad schematic)
At the start: 122 parts, among them SW10 SW_Push, SW11 SW_Push, SW14 SW_Push, SW15 SW_Push, SW16 SW_Push, SW18 SW_Push, SW20 SW_Push, SW21 SW_Push, SW22 SW_Push, SW23 SW_Push, SW24 SW_Push, SW25 SW_Push, SW26 SW_Push, SW27 SW_Push, SW28 SW_Push, SW29 SW_Push, SW3 SW_Push, SW30 SW_Push, SW31 SW_Push, SW32 SW_Push, SW35 SW_Push, SW36 SW_Push, SW37 SW_Push, SW38 SW_Push, SW39 SW_Push, SW40 SW_Push, SW41 SW_Push, SW42 SW_Push, SW43 SW_Push, SW44 SW_Push, SW45 SW_Push, SW46 SW_Push, SW47 SW_Push, SW48 SW_Push, SW49 SW_Push, SW5 SW_Push, SW50 SW_Push, SW51 SW_Push, SW52 SW_Push, SW53 SW_Push, SW54 SW_Push, SW56 SW_Push, SW58 SW_Push, SW59 SW_Push, SW60 SW_Push, SW61 SW_Push, SW62 SW_Push, SW65 SW_Push, SW66 SW_Push, SW67 SW_Push, SW68 SW_Push, SW7 SW_Push, SW71 SW_Push, SW73 SW_Push, SW74 SW_Push, SW76 SW_Push, SW79 SW_Push, SW82 SW_Push, SW84 SW_Push, SW86 SW_Push, SW9 SW_Push

Commit message: update keyswitch foodpoint
Parts:
- SW10, SW11, SW14, SW15, SW16, SW18, SW20, SW21, SW22, SW23, SW24, SW25, SW26, SW27, SW28, SW29, SW3, SW30, SW31, SW32, SW35, SW36, SW37, SW38, SW39, SW40, SW41, SW42, SW43, SW44, SW45, SW46, SW47, SW48, SW49, SW5, SW50, SW51, SW52, SW53, SW54, SW56, SW58, SW59, SW60, SW61, SW62, SW65, SW66, SW67, SW68, SW7, SW71, SW73, SW74, SW76, SW79, SW82, SW84, SW86, SW9: footprint keyswitches:Kailh_socket_MX -> Keyboard_Hotswap_Kailh:SW_Hotswap_Kailh_MX
Connections:
- net col1: now also SW10.1, SW3.1, SW5.1, SW7.1, SW9.1; no longer SW10.2, SW3.2, SW5.2, SW7.2, SW9.2
- net col10: now also SW51.1, SW52.1, SW53.1, SW54.1; no longer SW51.2, SW52.2, SW53.2, SW54.2
- net col11: now also SW56.1, SW58.1, SW59.1, SW60.1, SW61.1; no longer SW56.2, SW58.2, SW59.2, SW60.2, SW61.2
- net col12: now also SW62.1, SW65.1, SW66.1, SW67.1, SW68.1; no longer SW62.2, SW65.2, SW66.2, SW67.2, SW68.2
- net col13: now also SW71.1, SW73.1, SW74.1; no longer SW71.2, SW73.2, SW74.2
- net col14: now also SW76.1, SW79.1, SW82.1, SW84.1, SW86.1; no longer SW76.2, SW79.2, SW82.2, SW84.2, SW86.2
- net col2: now also SW11.1, SW14.1, SW15.1, SW16.1; no longer SW11.2, SW14.2, SW15.2, SW16.2
- net col3: now also SW18.1, SW20.1, SW21.1, SW22.1, SW23.1; no longer SW18.2, SW20.2, SW21.2, SW22.2, SW23.2
- net col4: now also SW24.1, SW25.1, SW26.1, SW27.1; no longer SW24.2, SW25.2, SW26.2, SW27.2
- net col5: now also SW28.1, SW29.1, SW30.1, SW31.1; no longer SW28.2, SW29.2, SW30.2, SW31.2
- net col6: now also SW35.1, SW36.1, SW37.1, SW38.1; no longer SW35.2, SW36.2, SW37.2, SW38.2
- net col7: now also SW32.1, SW39.1, SW40.1, SW41.1, SW42.1; no longer SW32.2, SW39.2, SW40.2, SW41.2, SW42.2
- net col8: now also SW43.1, SW44.1, SW45.1, SW46.1; no longer SW43.2, SW44.2, SW45.2, SW46.2
- net col9: now also SW47.1, SW48.1, SW49.1, SW50.1; no longer SW47.2, SW48.2, SW49.2, SW50.2
- net at D6.2 (A): now also SW7.2; no longer SW7.1
- net at D51.2 (A): now also SW59.2; no longer SW59.1
- net at D37.2 (A): now also SW44.2; no longer SW44.1
- net at D23.2 (A): now also SW28.2; no longer SW28.1
- net at D7.2 (A): now also SW9.2; no longer SW9.1
- net at D42.2 (A): now also SW49.2; no longer SW49.1
- net at D56.2 (A): now also SW66.2; no longer SW66.1
- net at D14.2 (A): now also SW18.2; no longer SW18.1
- net at D33.2 (A): now also SW40.2; no longer SW40.1
- net at D53.2 (A): now also SW61.2; no longer SW61.1
- net at D21.2 (A): now also SW26.2; no longer SW26.1
- net at D38.2 (A): now also SW45.2; no longer SW45.1
- net at D8.2 (A): now also SW10.2; no longer SW10.1
- net at D52.2 (A): now also SW60.2; no longer SW60.1
- net at D54.2 (A): now also SW62.2; no longer SW62.1
- net at D19.2 (A): now also SW24.2; no longer SW24.1
- net at D17.2 (A): now also SW22.2; no longer SW22.1
- net at D68.2 (A): now also SW86.2; no longer SW86.1
- net at D25.2 (A): now also SW30.2; no longer SW30.1
- net at D44.2 (A): now also SW51.2; no longer SW51.1
- net at D47.2 (A): now also SW54.2; no longer SW54.1
- net at D64.2 (A): now also SW76.2; no longer SW76.1
- net at D62.2 (A): now also SW74.2; no longer SW74.1
- net at D29.2 (A): now also SW36.2; no longer SW36.1
- net at D11.2 (A): now also SW15.2; no longer SW15.1
- net at D5.2 (A): now also SW5.2; no longer SW5.1
- net at D26.2 (A): now also SW31.2; no longer SW31.1
- net at D16.2 (A): now also SW21.2; no longer SW21.1
- net at D41.2 (A): now also SW48.2; no longer SW48.1
- net at D40.2 (A): now also SW47.2; no longer SW47.1
- net at D10.2 (A): now also SW14.2; no longer SW14.1
- net at D31.2 (A): now also SW38.2; no longer SW38.1
- net at D18.2 (A): now also SW23.2; no longer SW23.1
- net at D65.2 (A): now also SW79.2; no longer SW79.1
- net at D22.2 (A): now also SW27.2; no longer SW27.1
- net at D34.2 (A): now also SW41.2; no longer SW41.1
- net at D9.2 (A): now also SW11.2; no longer SW11.1
- net at D45.2 (A): now also SW52.2; no longer SW52.1
- net at D46.2 (A): now also SW53.2; no longer SW53.1
- net at D57.2 (A): now also SW67.2; no longer SW67.1
- net at D67.2 (A): now also SW82.2; no longer SW82.1
- net at D4.2 (A): now also SW3.2; no longer SW3.1
- net at D49.2 (A): now also SW56.2; no longer SW56.1
- net at D66.2 (A): now also SW84.2; no longer SW84.1
- net at D60.2 (A): now also SW71.2; no longer SW71.1
- net at D43.2 (A): now also SW50.2; no longer SW50.1
- net at D28.2 (A): now also SW35.2; no longer SW35.1
- net at D15.2 (A): now also SW20.2; no longer SW20.1
- net at D61.2 (A): now also SW73.2; no longer SW73.1
- net at D32.2 (A): now also SW39.2; no longer SW39.1
- net at D12.2 (A): now also SW16.2; no longer SW16.1
- net at D27.2 (A): now also SW32.2; no longer SW32.1
- net at D30.2 (A): now also SW37.2; no longer SW37.1
- net at D39.2 (A): now also SW46.2; no longer SW46.1
- net at D50.2 (A): now also SW58.2; no longer SW58.1
- net at D55.2 (A): now also SW65.2; no longer SW65.1
- net at D36.2 (A): now also SW43.2; no longer SW43.1
- net at D20.2 (A): now also SW25.2; no longer SW25.1
- net at D24.2 (A): now also SW29.2; no longer SW29.1
- net at D35.2 (A): now also SW42.2; no longer SW42.1
- net at D58.2 (A): now also SW68.2; no longer SW68.1
Other:
- moved on the sheet: SW10, SW11, SW14, SW15, SW16, SW18, SW20, SW21, SW22, SW23, SW24, SW25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
